File: hardware/thermostat-carrier/thermostat-carrier.kicad_sch (KiCad schematic)
At the start: 82 parts, among them J1 24 VAC, J2 Calls 24 VAC, J3 USB-C 5 V in, J4 USB-A 5 V to display, J5 Display I2C, J6 Display IO6, J7 Room SHT45 (Qwiic), K1 AQV252G, K2 AQV252G, K3 AQV252G, K4 AQV252G, K5 AQV252G, K6 AQV252G, U1 LM2596HV, U10 H11AA1, U11 H11AA1, U12 H11AA1, U2 AMS1117-3.3, U3 MCP23017-E/SO, U4 TPS3823-33, U5 SC18IS602B, U6 Wio-SX1262, U7 H11AA1, U8 H11AA1, U9 H11AA1

Commit message: Thermostat carrier: stack behind the Waveshare 4.3 on its own outline
The carrier now matches the display's 106 x 68 mm outline and screws to its
four M2.5 standoffs (measured from Waveshare's STEP model). SMD parts sit on
the wall side for JLC assembly; a right-edge notch clears the display's side
sockets, and short HY2.0 leads go to J5 (I2C) and J6 (IO6 for LoRa DIO1).

- Power: TPS54360B buck to 5.3 V replaces the LM2596 module; USB-C in for
  display-only use, USB-C out carries 5 V to the display.
- route.py: fan-out vias stay inside the outline and off exposed pads;
  pour islands are joined by vias, short bridges or a grid search
  (maze_bridge) for a GND track.
- gen_sch: PWR_FLAG on label nets (flag_nets) for the buck's VRAW input.
- make_fab: all-SMD JLC CPL/BOM for the thermostat carrier.
- DRC 0 violations, 0 unconnected, schematic parity clean; ERC clean.

Co-Authored-By: Claude Opus 5.5 <noreply@anthropic.com>
Claude-Session: https://claude.ai/code/session_011hFUPCDAe7urxnoDwvZQtt
Parts:
- removed C3: 220µF 16V, Capacitor_THT:CP_Radial_D6.3mm_P2.50mm, symbol Device:C_Polarized
- removed C4: 10µF 16V, Capacitor_THT:CP_Radial_D5.0mm_P2.00mm, symbol Device:C_Polarized
- removed C5: 22µF 10V, Capacitor_THT:CP_Radial_D5.0mm_P2.00mm, symbol Device:C_Polarized
- removed J4: USB-A 5 V to display, Connector_USB:USB_A_Molex_67643_Horizontal, symbol Connector:USB_A
- removed J5: Display I2C, Connector_PinHeader_2.54mm:PinHeader_1x04_P2.54mm_Vertical, symbol Connector_Generic:Conn_01x04
- removed J6: Display IO6, Connector_PinHeader_2.54mm:PinHeader_1x03_P2.54mm_Vertical, symbol Connector_Generic:Conn_01x03
- removed U1: LM2596HV, hvac_carrier:LM2596HVS_Module, symbol hvac_carrier:LM2596HV_Module
- added C11: 0.1µF, Capacitor_SMD:C_0805_2012Metric, symbol Device:C
- added C12: 22nF, Capacitor_SMD:C_0805_2012Metric, symbol Device:C
- added C13: 100pF, Capacitor_SMD:C_0805_2012Metric, symbol Device:C
- added C14, C15, C3: 22µF 16V, Capacitor_SMD:C_1206_3216Metric, symbol Device:C
- added C4: 10µF 25V, Capacitor_SMD:C_0805_2012Metric, symbol Device:C
- added C5: 22µF 10V, Capacitor_SMD:C_0805_2012Metric, symbol Device:C
- added D11: SS36, Diode_SMD:D_SMA, symbol Device:D_Schottky
- added J4: USB-C 5 V to display, Connector_USB:USB_C_Receptacle_GCT_USB4125-xx-x_6P_TopMnt_Horizontal, symbol Connector:USB_C_Receptacle_PowerOnly_6P
- added J5: Display I2C, Connector_JST:JST_PH_B4B-PH-SM4-TB_1x04-1MP_P2.00mm_Vertical, symbol Connector_Generic_MountingPin:Conn_01x04_MountingPin
- added J6: Display IO6, Connector_JST:JST_PH_B3B-PH-SM4-TB_1x03-1MP_P2.00mm_Vertical, symbol Connector_Generic_MountingPin:Conn_01x03_MountingPin
- added L1: 22µH 2A, Inductor_SMD:L_7.3x7.3_H4.5, symbol Device:L
- added R30: 243k, Resistor_SMD:R_0805_2012Metric, symbol Device:R
- added R31, R34, R35: 56k, Resistor_SMD:R_0805_2012Metric, symbol Device:R
- added R32: 10k, Resistor_SMD:R_0805_2012Metric, symbol Device:R
- added R33: 6.8k, Resistor_SMD:R_0805_2012Metric, symbol Device:R
- added U1: TPS54360BDDAR, Package_SO:TI_SO-PowerPAD-8_ThermalVias, symbol Regulator_Switching:TPS54360DDA
- C1: value 1000µF 63V -> 220µF 63V; footprint Capacitor_THT:CP_Radial_D12.5mm_P5.00mm -> Capacitor_SMD:CP_Elec_10x10.5
- C10, C6, C7, C8, C9: footprint Capacitor_SMD:C_0805_2012Metric_Pad1.18x1.45mm_HandSolder -> Capacitor_SMD:C_0805_2012Metric
- C2: value 0.1µF -> 2.2µF 100V; footprint Capacitor_THT:C_Disc_D5.0mm_W2.5mm_P2.50mm -> Capacitor_SMD:C_1210_3225Metric
- D1: value SMBJ48CA -> SMBJ40CA; footprint Diode_SMD:D_SMB_Handsoldering -> Diode_SMD:D_SMB
- D10, D5, D6, D7, D8, D9: footprint Diode_SMD:D_SMB_Handsoldering -> Diode_SMD:D_SMB
- D2: value 1N4007 -> S1M; footprint Diode_THT:D_DO-41_SOD81_P10.16mm_Horizontal -> Diode_SMD:D_SMA
- D3, D4: footprint Diode_SMD:D_SMA_Handsoldering -> Diode_SMD:D_SMA
- F1: value 0.5 A fast -> 0.5 A fast 63 V; footprint Fuse:Fuseholder_Clip-5x20mm_Littelfuse_111_Inline_P20.00x5.00mm_D1.05mm_Horizontal -> Fuse:Fuse_1206_3216Metric
- F2, F3: value 0ZRE0125FF -> 2920L110/60; footprint Fuse:Fuse_BelFuse_0ZRE0125FF_L21.2mm_W5.3mm -> Fuse:Fuse_2920_7451Metric
- H1, H2, H3, H4: value M3 -> M2.5; footprint MountingHole:MountingHole_3.2mm_M3_DIN965 -> MountingHole:MountingHole_2.7mm_M2.5_DIN965
- J1: footprint Connector_Phoenix_MC_HighVoltage:PhoenixContact_MC_1,5_3-G-5.08_1x03_P5.08mm_Horizontal -> Connector_Phoenix_MC:PhoenixContact_MCV_1,5_3-G-3.5_1x03_P3.50mm_Vertical
- J2: footprint Connector_Phoenix_MC_HighVoltage:PhoenixContact_MC_1,5_6-G-5.08_1x06_P5.08mm_Horizontal -> Connector_Phoenix_MC:PhoenixContact_MCV_1,5_6-G-3.5_1x06_P3.50mm_Vertical
- K1, K2, K3, K4, K5, K6: value AQV252G -> AQV252GS; footprint Package_DIP:DIP-6_W7.62mm_Socket -> Package_DIP:SMDIP-6_W9.53mm
- R1, R10, R11, R12, R13, R14, R2, R21, R22, R23, R24, R25, R26, R27, R28, R29, R3, R4, R5, R6, R7, R8, R9: footprint Resistor_SMD:R_0805_2012Metric_Pad1.20x1.40mm_HandSolder -> Resistor_SMD:R_0805_2012Metric
- R15, R16, R17, R18, R19, R20: value 4.7k ½W -> 4.7k 2010; footprint Resistor_THT:R_Axial_DIN0309_L9.0mm_D3.2mm_P12.70mm_Horizontal -> Resistor_SMD:R_2010_5025Metric
- U10, U11, U12, U7, U8, U9: value H11AA1 -> H11AA1SM; footprint Package_DIP:DIP-6_W7.62mm_Socket -> Package_DIP:SMDIP-6_W9.53mm
- U4: footprint Package_TO_SOT_SMD:SOT-23-5_HandSoldering -> Package_TO_SOT_SMD:SOT-23-5
Connections:
- net +3V3: now also C5.1
- net +5V: now also C3.1, C4.1, J4.A9 (VBUS), J4.B9 (VBUS), R34.1, R35.1
- net GND: now also C12.2, C13.2, C14.2, C15.2, C3.2, C4.2, C5.2, D11.2 (A), J4.A12 (GND), J4.B12 (GND), J4.SH (SHIELD), J5.2 (Pin_2), J5.MP (MountPin), J6.2 (Pin_2), J6.MP (MountPin), R30.2, R32.2, U1.7 (GND), U1.9 (GNDPAD)
- net LORA_DIO1: now also J6.3 (Pin_3)
- net SCL: now also J5.4 (Pin_4)
- net SDA: now also J5.3 (Pin_3)
- net V5_BUCK: now also C14.1, C15.1, L1.2, R31.1
- net VRAW: now also U1.2 (VIN)
- new net BOOT: C11.1, U1.1 (BOOT)
- new net CCO1: J4.A5 (CC1), R34.2
- new net CCO2: J4.B5 (CC2), R35.2
- new net COMP: C13.1, R33.1, U1.6 (COMP)
- new net COMP_RC: C12.1, R33.2
- new net FB: R31.2, R32.1, U1.5 (FB)
- new net RT: R30.1, U1.4 (RT/CLK)
- new net SW: C11.2, D11.1 (K), L1.1, U1.8 (SW)
- no-connect marks 37 -> 36
Other:
- note added: "A Power: Rc-C 24 VAC (TPS54360B buck) or USB-C 5 V in; USB-C 5 V out to the display"
- note removed: "A Power: Rc-C 24 VAC or USB-C 5 V; USB-A 5 V to the display"
